File: Audio Power Supply Board v3.0/Aux.kicad_sch (KiCad schematic)
At the start: 6 parts

Commit message: Change to a modular drawing and design
Parts:
- renumbered C5 to C31, D4 to D22, D5 to D23, D6 to D24, D7 to D25
Changed lines of the file:
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@@
   (symbol (lib_id "power:PWR_FLAG") (at 107.315 84.455 0) (unit 1)
     (in_bom yes) (on_board yes)
-    (property "Reference" "#FLG0103" (id 0) (at 107.315 82.55 0)
+    (property "Reference" "#FLG07" (id 0) (at 107.315 82.55 0)
       (effects (font (size 1.27 1.27)) hide)
     )
@@
   (symbol (lib_id "power:PWR_FLAG") (at 107.315 92.075 0) (unit 1)
     (in_bom yes) (on_board yes)
-    (property "Reference" "#FLG0102" (id 0) (at 107.315 90.17 0)
+    (property "Reference" "#FLG08" (id 0) (at 107.315 90.17 0)
       (effects (font (size 1.27 1.27)) hide)
     )
@@
   (symbol (lib_id "Device:C_Polarized_Small") (at 93.345 88.265 0) (unit 1)
     (in_bom yes) (on_board yes)
-    (property "Reference" "C5" (id 0) (at 95.5041 87.5041 0)
+    (property "Reference" "C31" (id 0) (at 95.5041 87.5041 0)
       (effects (font (size 1.27 1.27)) (justify left))
     )
@@
   (symbol (lib_id "Diode:1N4004") (at 57.15 75.565 90) (unit 1)
     (in_bom yes) (on_board yes)
-    (property "Reference" "D4" (id 0) (at 59.1821 74.8041 90)
+    (property "Reference" "D22" (id 0) (at 59.1821 74.8041 90)
       (effects (font (size 1.27 1.27)) (justify right))
     )
@@
   (symbol (lib_id "Diode:1N4004") (at 57.15 97.155 90) (mirror x) (unit 1)
     (in_bom yes) (on_board yes)
-    (property "Reference" "D5" (id 0) (at 59.1821 97.9159 90)
+    (property "Reference" "D23" (id 0) (at 59.1821 97.9159 90)
       (effects (font (size 1.27 1.27)) (justify right))
     )
@@
   (symbol (lib_id "Diode:1N4004") (at 70.485 75.565 90) (mirror x) (unit 1)
     (in_bom yes) (on_board yes)
-    (property "Reference" "D6" (id 0) (at 72.5171 76.3259 90)
+    (property "Reference" "D24" (id 0) (at 72.5171 76.3259 90)
       (effects (font (size 1.27 1.27)) (justify right))
     )
@@
   (symbol (lib_id "Diode:1N4004") (at 70.485 97.155 90) (unit 1)
     (in_bom yes) (on_board yes)
-    (property "Reference" "D7" (id 0) (at 72.5171 96.3941 90)
+    (property "Reference" "D25" (id 0) (at 72.5171 96.3941 90)
       (effects (font (size 1.27 1.27)) (justify right))
     )
