File: Audio Power Supply Board v3.0/Controller.kicad_sch (KiCad schematic)
At the start: 1 part, among them J2 CON_CTRL_Board

Commit message: Change to a modular drawing and design
Parts:
- J13: renamed from J2; symbol Power-Supply-Board-v2.0-rescue:Conn_01x14-Connector_Generic -> Connector_Generic:Conn_01x14
Connections:
- net GNDA renamed GND
- net HO renamed Ho
Changed lines of the file:
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@@
 (kicad_sch (version 20210126) (generator eeschema)
   (paper "A4")
-  (junction (at 116.84 107.315) (diameter 0.9144) (color 0 0 0 0))
   (no_connect (at 120.65 76.835))
   (no_connect (at 120.65 84.455))
@@
     (stroke (width 0) (type solid) (color 0 0 0 0))
   )
-  (wire (pts (xy 108.585 107.315) (xy 116.84 107.315))
-    (stroke (width 0) (type solid) (color 0 0 0 0))
-  )
-  (wire (pts (xy 116.84 107.315) (xy 116.84 112.395))
-    (stroke (width 0) (type solid) (color 0 0 0 0))
-  )
-  (wire (pts (xy 116.84 107.315) (xy 120.65 107.315))
+  (wire (pts (xy 108.585 107.315) (xy 120.65 107.315))
     (stroke (width 0) (type solid) (color 0 0 0 0))
   )
@@
     (effects (font (size 1.27 1.27)) (justify right))
   )
-  (hierarchical_label "HO" (shape input) (at 108.585 79.375 180)
+  (hierarchical_label "Ho" (shape input) (at 108.585 79.375 180)
     (effects (font (size 1.27 1.27)) (justify right))
   )
@@
     (effects (font (size 1.27 1.27)) (justify right))
   )
-  (symbol (lib_id "Power-Supply-Board-v2.0-rescue:GNDA-power") (at 116.84 112.395 0) (unit 1)
+  (symbol (lib_id "Connector_Generic:Conn_01x14") (at 125.73 89.535 0) (unit 1)
     (in_bom yes) (on_board yes)
-    (property "Reference" "#PWR04" (id 0) (at 116.84 118.745 0)
-      (effects (font (size 1.27 1.27)) hide)
-    )
-    (property "Value" "GNDA" (id 1) (at 116.967 116.7892 0))
-    (property "Footprint" "" (id 2) (at 116.84 112.395 0)
-      (effects (font (size 1.27 1.27)) hide)
-    )
-    (property "Datasheet" "" (id 3) (at 116.84 112.395 0)
-      (effects (font (size 1.27 1.27)) hide)
-    )
-    (pin "1")
-  )
-  (symbol (lib_id "Power-Supply-Board-v2.0-rescue:Conn_01x14-Connector_Generic") (at 125.73 89.535 0) (unit 1)
-    (in_bom yes) (on_board yes)
-    (property "Reference" "J2" (id 0) (at 121.92 67.945 0)
+    (property "Reference" "J13" (id 0) (at 121.92 67.945 0)
       (effects (font (size 1.27 1.27)) (justify left))
     )
@@
       (effects (font (size 1.27 1.27)) (justify left))
     )
-    (property "Footprint" "Connector_PinSocket_2.54mm:PinSocket_1x14_P2.54mm_Vertical" (id 2) (at -269.24 291.465 0)
+    (property "Footprint" "Connector_PinSocket_2.54mm:PinSocket_1x14_P2.54mm_Vertical" (id 2) (at 125.73 89.535 0)
       (effects (font (size 1.27 1.27)) hide)
     )
-    (property "Datasheet" "" (id 3) (at -269.24 291.465 0)
+    (property "Datasheet" "~" (id 3) (at 125.73 89.535 0)
       (effects (font (size 1.27 1.27)) hide)
     )
