File: Audio Power Supply Board v3.0/FanCtrl.kicad_sch (KiCad schematic)
At the start: 0 parts

Commit message: Change to a modular drawing and design
Parts:
- added C23: 1/50, Capacitor_THT:CP_Radial_D8.0mm_P2.50mm, symbol Device:C_Polarized
- added C24: 10n, Capacitor_THT:C_Rect_L4.6mm_W3.8mm_P2.50mm_MKS02_FKP02, symbol Device:C_Small
- added C25: 4.7µ/50, Capacitor_THT:CP_Radial_D5.0mm_P2.00mm, symbol Device:C_Polarized
- added D15: 15V, Diode_THT:D_DO-15_P12.70mm_Horizontal, symbol Device:D_Zener
- added D16: 1N4148, Diode_THT:D_DO-35_SOD27_P7.62mm_Horizontal, symbol Diode:1N4148
- added D17: 8V2, Diode_THT:D_DO-15_P12.70mm_Horizontal, symbol Device:D_Zener
- added Q2, Q4, Q5: MPSA56, Package_TO_SOT_THT:TO-92_Wide, symbol Power-Supply-Board-v2.0-rescue:MPSA56-Power-Supply-Board-v1.0-rescue
- added Q3: MPSA06, TO_SOT_Packages_THT:TO-92_Molded_Narrow, symbol Userlibrary:MPSA06
- added Q6: MJE350, Package_TO_SOT_THT:TO-126-3_Vertical, symbol Device:Q_PNP_ECB
- added R10: 18k, Resistor_THT:R_Axial_DIN0204_L3.6mm_D1.6mm_P7.62mm_Horizontal, symbol Device:R
- added R11, R8: 220, Resistor_THT:R_Axial_DIN0204_L3.6mm_D1.6mm_P7.62mm_Horizontal, symbol Device:R
- added R4: 8k2, Resistor_THT:R_Axial_DIN0204_L3.6mm_D1.6mm_P7.62mm_Horizontal, symbol Device:R
- added R5: 5k6, Resistor_THT:R_Axial_DIN0204_L3.6mm_D1.6mm_P7.62mm_Horizontal, symbol Device:R
- added R6, R7: 330, Resistor_THT:R_Axial_DIN0204_L3.6mm_D1.6mm_P7.62mm_Horizontal, symbol Device:R
- added R9: 12k, Resistor_THT:R_Axial_DIN0204_L3.6mm_D1.6mm_P7.62mm_Horizontal, symbol Device:R
Connections:
- new net: C23.2, D15.2 (A), Q2.2 (B), R4.2
- new net: Q5.2 (B), R11.1
- new net: C24.2, D17.2 (A), Q4.3 (C), R10.2, R11.2, R9.2
- new net: D16.1 (K), Q3.2 (B)
- new net: Q5.1 (E), Q6.3 (B)
- new net: D17.1 (K), Q3.1 (E)
- new net: Q3.3 (C), R8.1
- new net: C24.1, Q4.2 (B), R7.1
- new net: Q2.1 (E), R5.1
- new net -24V: Q2.3 (C), Q5.3 (C), Q6.2 (C), R10.1, R4.1, R9.1
- new net FAN-: C25.1, Q6.1 (E)
- new net GND: C23.1, C25.2, D15.1 (K), Q4.1 (E), R6.2, R8.2
- new net PAH1: R6.1, R7.2
- new net PAH2: D16.2 (A), R5.2
