File: Audio Power Supply Board v3.0/FanCtrl.kicad_sch (KiCad schematic)
At the start: 19 parts, among them Q2 MPSA56, Q3 MPSA06, Q4 MPSA56, Q5 MPSA56, Q6 MJE350

Commit message: Add protection circuits
Parts:
- Q2, Q4, Q5: footprint Package_TO_SOT_THT:TO-92_Wide -> Package_TO_SOT_THT:TO-92_Inline; symbol Power-Supply-Board-v2.0-rescue:MPSA56-Power-Supply-Board-v1.0-rescue -> Transistor_BJT:MPSA42
Changed lines of the file:
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@@
     (pin "2")
   )
-  (symbol (lib_id "Power-Supply-Board-v2.0-rescue:MPSA56-Power-Supply-Board-v1.0-rescue") (at 102.87 106.045 0) (mirror x) (unit 1)
+  (symbol (lib_id "Transistor_BJT:MPSA42") (at 102.87 106.045 0) (mirror x) (unit 1)
     (in_bom yes) (on_board yes)
     (property "Reference" "Q2" (id 0) (at 107.7214 104.8766 0)
@@
       (effects (font (size 1.27 1.27)) (justify left))
     )
-    (property "Footprint" "Package_TO_SOT_THT:TO-92_Wide" (id 2) (at -261.62 -37.465 0)
-      (effects (font (size 1.27 1.27)) hide)
+    (property "Footprint" "Package_TO_SOT_THT:TO-92_Inline" (id 2) (at 107.95 104.14 0)
+      (effects (font (size 1.27 1.27) italic) (justify left) hide)
     )
-    (property "Datasheet" "" (id 3) (at -266.7 -40.005 0)
-      (effects (font (size 1.27 1.27)) hide)
+    (property "Datasheet" "http://www.onsemi.com/pub_link/Collateral/MPSA42-D.PDF" (id 3) (at 102.87 106.045 0)
+      (effects (font (size 1.27 1.27)) (justify left) hide)
     )
     (pin "1")
@@
     (pin "3")
   )
-  (symbol (lib_id "Power-Supply-Board-v2.0-rescue:MPSA56-Power-Supply-Board-v1.0-rescue") (at 140.97 71.755 0) (mirror x) (unit 1)
+  (symbol (lib_id "Transistor_BJT:MPSA42") (at 140.97 71.755 0) (mirror x) (unit 1)
     (in_bom yes) (on_board yes)
     (property "Reference" "Q4" (id 0) (at 145.8214 70.5866 0)
@@
       (effects (font (size 1.27 1.27)) (justify left))
     )
-    (property "Footprint" "Package_TO_SOT_THT:TO-92_Wide" (id 2) (at -223.52 -71.755 0)
-      (effects (font (size 1.27 1.27)) hide)
+    (property "Footprint" "Package_TO_SOT_THT:TO-92_Inline" (id 2) (at 146.05 69.85 0)
+      (effects (font (size 1.27 1.27) italic) (justify left) hide)
     )
-    (property "Datasheet" "" (id 3) (at -228.6 -74.295 0)
-      (effects (font (size 1.27 1.27)) hide)
+    (property "Datasheet" "http://www.onsemi.com/pub_link/Collateral/MPSA42-D.PDF" (id 3) (at 140.97 71.755 0)
+      (effects (font (size 1.27 1.27)) (justify left) hide)
     )
     (pin "1")
@@
     (pin "3")
   )
-  (symbol (lib_id "Power-Supply-Board-v2.0-rescue:MPSA56-Power-Supply-Board-v1.0-rescue") (at 161.29 106.045 0) (mirror x) (unit 1)
+  (symbol (lib_id "Transistor_BJT:MPSA42") (at 161.29 106.045 0) (mirror x) (unit 1)
     (in_bom yes) (on_board yes)
     (property "Reference" "Q5" (id 0) (at 166.1414 104.8766 0)
@@
       (effects (font (size 1.27 1.27)) (justify left))
     )
-    (property "Footprint" "Package_TO_SOT_THT:TO-92_Wide" (id 2) (at -203.2 -37.465 0)
-      (effects (font (size 1.27 1.27)) hide)
+    (property "Footprint" "Package_TO_SOT_THT:TO-92_Inline" (id 2) (at 166.37 104.14 0)
+      (effects (font (size 1.27 1.27) italic) (justify left) hide)
     )
-    (property "Datasheet" "" (id 3) (at -208.28 -40.005 0)
-      (effects (font (size 1.27 1.27)) hide)
+    (property "Datasheet" "http://www.onsemi.com/pub_link/Collateral/MPSA42-D.PDF" (id 3) (at 161.29 106.045 0)
+      (effects (font (size 1.27 1.27)) (justify left) hide)
     )
     (pin "1")
