File: Audio Power Supply Board v3.0/Mute.kicad_sch (KiCad schematic)
At the start: 0 parts

Commit message: Change to a modular drawing and design
Parts:
- added C26: 470µ/35, Capacitor_THT:CP_Radial_D8.0mm_P3.50mm, symbol Device:C_Polarized
- added C27: 100n, Capacitor_THT:C_Rect_L9.0mm_W4.0mm_P7.50mm_MKT, symbol Device:C_Small
- added C28: 33µ/35, Capacitor_THT:CP_Radial_D5.0mm_P2.00mm, symbol Device:C_Polarized
- added D18: 1N4148, Diode_THT:D_DO-35_SOD27_P7.62mm_Horizontal, symbol Diode:1N4148
- added D19: 15V, Diode_THT:D_DO-15_P12.70mm_Horizontal, symbol Device:D_Zener
- added Q10, Q7, Q8: BC546, Package_TO_SOT_THT:TO-92_Inline, symbol Transistor_BJT:BC546
- added Q9: MPSA56, Package_TO_SOT_THT:TO-92_Inline, symbol Transistor_BJT:MPSA92
- added R12: 4k7, Resistor_THT:R_Axial_DIN0204_L3.6mm_D1.6mm_P7.62mm_Horizontal, symbol Device:R
- added R13: 150k, Resistor_THT:R_Axial_DIN0204_L3.6mm_D1.6mm_P7.62mm_Horizontal, symbol Device:R
- added R14, R16, R17: 220k, Resistor_THT:R_Axial_DIN0204_L3.6mm_D1.6mm_P7.62mm_Horizontal, symbol Device:R
- added R15: 100k, Resistor_THT:R_Axial_DIN0204_L3.6mm_D1.6mm_P7.62mm_Horizontal, symbol Device:R
- added R18: 56k, Resistor_THT:R_Axial_DIN0204_L3.6mm_D1.6mm_P7.62mm_Horizontal, symbol Device:R
Connections:
- new net: Q8.1 (C), R17.2
- new net: Q7.1 (C), Q8.2 (B), R14.2, R15.1
- new net: D19.2 (A), Q7.2 (B)
- new net: C28.1, D18.2 (A), D19.1 (K), Q10.1 (C), R13.2
- new net: Q9.2 (B), R16.2, R17.1
- new net GND: C26.2, C27.2, C28.2, Q10.3 (E), Q7.3 (E), Q8.3 (E), R12.2, R15.2, R18.2
- new net MUTE: Q9.3 (C)
- new net MUTEIN: Q10.2 (B), R18.1
- new net V+1: C26.1, Q9.1 (E), R13.1, R14.1, R16.1
- new net V+2: C27.1, D18.1 (K), R12.1
