File: Audio Power Supply Board v3.0/Power.kicad_sch (KiCad schematic)
At the start: 0 parts

Commit message: Change to a modular drawing and design
Parts:
- added C29, C30: 27n/300V, Capacitor_THT:C_Rect_L19.0mm_W6.0mm_P15.00mm_MKS4, symbol Device:C
- added D20, D21: 1N4148, Diode_THT:D_DO-35_SOD27_P7.62mm_Horizontal, symbol Diode:1N4148
- added HS3: Heatsink, UserLibrary:Heatsink_100x45x18mm_3xFixationM3, symbol Power-Supply-Board-v2.0-rescue:Heatsink-Mechanical
- added L6: 53100C-I-XFR, SamacSys_Parts:53100C, symbol Userlibrary:53100C-I-XFR
- added Q11, Q12: IRFP460, Package_TO_SOT_THT:TO-220-3_Vertical, symbol Transistor_FET:IRF540N
- added R19, R20: 10, Resistor_THT:R_Axial_DIN0204_L3.6mm_D1.6mm_P7.62mm_Horizontal, symbol Device:R
- added R21, R22: 1k, Resistor_THT:R_Axial_DIN0204_L3.6mm_D1.6mm_P7.62mm_Horizontal, symbol Device:R
Connections:
- new net: C29.1, C30.2, L6.8 (PRI2)
- new net: D20.2 (A), Q11.1 (G), R19.1, R21.1
- new net: D21.2 (A), Q12.1 (G), R20.1, R22.1
- new net +Vb: Q11.2 (D)
- new net CS+: L6.3 (SEC2)
- new net CS-: L6.1 (SEC1)
- new net GND: Q12.3 (S), R22.2
- new net Ho: D20.1 (K), R19.2
- new net L1: Q11.3 (S), Q12.2 (D), R21.2
- new net L2: L6.7 (PRI1)
- new net Lo: D21.1 (K), R20.2
- new net V/2: C29.2, C30.1
