File: Audio Power Supply Board v3.0/Power.kicad_sch (KiCad schematic)
At the start: 12 parts, among them Q11 IRFP460, Q12 IRFP460

Commit message: Add protection circuits
Parts:
- HS3: symbol Power-Supply-Board-v2.0-rescue:Heatsink-Mechanical -> Mechanical:Heatsink
Changed lines of the file:
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@@
     (pin "2")
   )
-  (symbol (lib_id "Power-Supply-Board-v2.0-rescue:Heatsink-Mechanical") (at 185.42 78.105 0) (unit 1)
+  (symbol (lib_id "Mechanical:Heatsink") (at 185.42 78.105 0) (unit 1)
     (in_bom yes) (on_board yes)
     (property "Reference" "HS3" (id 0) (at 189.0268 75.0316 0)
