File: Audio Power Supply Board v3.0/Secondary Power.kicad_sch (KiCad schematic)
At the start: 0 parts

Commit message: Change to a modular drawing and design
Parts:
- added C15, C16: 470µ/35, Capacitor_THT:CP_Radial_D8.0mm_P3.50mm, symbol Device:C_Polarized
- added C17, C18: 47µ/35, Capacitor_THT:CP_Radial_D5.0mm_P2.50mm, symbol Device:C_Polarized
- added C19, C20: 10µ/35, Capacitor_THT:CP_Radial_D5.0mm_P2.50mm, symbol Device:C_Polarized
- added C21, C22: 470n, Capacitor_THT:C_Rect_L7.2mm_W11.0mm_P5.00mm_FKS2_FKP2_MKS2_MKP2, symbol Device:C_Small
- added D13, D14: 1N4001, Diode_THT:D_DO-35_SOD27_P7.62mm_Horizontal, symbol Diode:1N4148
- added HS1, HS2: Heatsink, Userlibrary:Heatsink EA2 T220, symbol Power-Supply-Board-v2.0-rescue:Heatsink-Mechanical
- added L4, L5: 10µ, Inductor_SMD:L_Wuerth_WE-PD-Typ-LS_Handsoldering, symbol Device:L_Ferrite
- added U1: LM7815ACT, Package_TO_SOT_THT:TO-220-3_Vertical, symbol Regulator_Linear:LM7815_TO220
- added U2: LM7915CT, Package_TO_SOT_THT:TO-220-3_Vertical, symbol Regulator_Linear:LM7915_TO220
Connections:
- new net +15V: C19.1, C22.1, D13.1 (K), U1.3 (VO)
- new net +24V: C17.1, L4.1, U1.1 (VI)
- new net -15V: C20.2, C21.1, D14.2 (A), U2.3 (VO)
- new net -24V: C18.2, L5.1, U2.2 (VI)
- new net GND: C15.2, C16.1, C17.2, C18.1, C19.2, C20.1, C21.2, C22.2, D13.2 (A), D14.1 (K), U1.2 (GND), U2.1 (GND)
- new net V+: C15.1, L4.2
- new net V-: C16.2, L5.2
