File: Audio Power Supply Board v3.0/Secondary Power.kicad_sch (KiCad schematic)
At the start: 16 parts, among them U1 LM7815ACT, U2 LM7915CT

Commit message: Add protection circuits
Parts:
- HS1, HS2: symbol Power-Supply-Board-v2.0-rescue:Heatsink-Mechanical -> Mechanical:Heatsink
Changed lines of the file:
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@@
   (symbol (lib_id "power:PWR_FLAG") (at 100.965 60.96 0) (unit 1)
     (in_bom yes) (on_board yes)
-    (property "Reference" "#FLG?" (id 0) (at 100.965 59.055 0)
+    (property "Reference" "#FLG04" (id 0) (at 100.965 59.055 0)
       (effects (font (size 1.27 1.27)) hide)
     )
@@
   (symbol (lib_id "power:PWR_FLAG") (at 100.965 95.25 180) (unit 1)
     (in_bom yes) (on_board yes)
-    (property "Reference" "#FLG?" (id 0) (at 100.965 97.155 0)
+    (property "Reference" "#FLG05" (id 0) (at 100.965 97.155 0)
       (effects (font (size 1.27 1.27)) hide)
     )
@@
   (symbol (lib_id "power:PWR_FLAG") (at 154.305 75.565 0) (unit 1)
     (in_bom yes) (on_board yes)
-    (property "Reference" "#FLG?" (id 0) (at 154.305 73.66 0)
+    (property "Reference" "#FLG06" (id 0) (at 154.305 73.66 0)
       (effects (font (size 1.27 1.27)) hide)
     )
@@
     (pin "1")
   )
-  (symbol (lib_id "Power-Supply-Board-v2.0-rescue:GND-power") (at 151.765 107.95 0) (unit 1)
+  (symbol (lib_id "power:GND") (at 151.765 107.95 0) (unit 1)
     (in_bom yes) (on_board yes)
     (property "Reference" "#PWR08" (id 0) (at 153.035 106.68 0)
@@
     )
     (property "Value" "GND" (id 1) (at 151.8666 106.0704 0))
-    (property "Footprint" "" (id 2) (at -235.585 223.52 0)
+    (property "Footprint" "" (id 2) (at 151.765 107.95 0)
       (effects (font (size 1.27 1.27)) hide)
     )
-    (property "Datasheet" "" (id 3) (at -235.585 223.52 0)
+    (property "Datasheet" "" (id 3) (at 151.765 107.95 0)
       (effects (font (size 1.27 1.27)) hide)
     )
@@
     (pin "2")
   )
-  (symbol (lib_id "Power-Supply-Board-v2.0-rescue:Heatsink-Mechanical") (at 120.015 36.83 0) (unit 1)
+  (symbol (lib_id "Mechanical:Heatsink") (at 120.015 36.83 0) (unit 1)
     (in_bom yes) (on_board yes)
     (property "Reference" "HS1" (id 0) (at 123.6218 33.7566 0)
@@
     )
   )
-  (symbol (lib_id "Power-Supply-Board-v2.0-rescue:Heatsink-Mechanical") (at 137.16 36.83 0) (unit 1)
+  (symbol (lib_id "Mechanical:Heatsink") (at 137.16 36.83 0) (unit 1)
     (in_bom yes) (on_board yes)
     (property "Reference" "HS2" (id 0) (at 140.7668 33.7566 0)
