File: Audio Power Supply Board v3.0/Protection.kicad_sch (KiCad schematic)
At the start: 0 parts

Commit message: Add protection circuits
Parts:
- added C37: 100p, symbol Device:C_Small
- added C38: 47uF/25V, symbol Device:C_Polarized_Small
- added C39: 10uF/50V, symbol Device:C_Polarized_Small
- added C40: C, symbol Device:C
- added D30: 1N4148, symbol Device:D
- added D32, D34, D35: D, symbol Device:D
- added D33: D_Zener, symbol Device:D_Zener
- added Q19, Q20, Q21, Q23, Q24, Q26: BC846, Package_TO_SOT_SMD:SOT-23, symbol Transistor_BJT:BC846
- added Q22: BC856, Package_TO_SOT_SMD:SOT-23, symbol Transistor_BJT:BC856
- added Q25, Q27, Q28: DTA114E, symbol Transistor_BJT:DTA114E
- added R36, R37: 120k, symbol Device:R
- added R38, R41, R45, R49: 10k, symbol Device:R
- added R39: 22k, symbol Device:R
- added R40, R43: 47k, symbol Device:R
- added R42: R, symbol Device:R
- added R44: 47kΩ, symbol Device:R
- added R46, R50: 56k, symbol Device:R
- added R47: 68k, symbol Device:R
- added R48: 1k2, symbol Device:R
- added R51: 6k8, symbol Device:R
- added R52, R53: 3k3, symbol Device:R
Connections:
- new net: Q28.3 (C), R53.1
- new net: D32.1 (K), R48.1
- new net: Q22.3 (C), R45.2, R46.2
- new net: D30.2 (A), Q21.3 (C), Q23.3 (C), R42.1
- new net: Q26.3 (C), Q27.1 (B)
- new net: Q27.3 (C), R52.1
- new net: D35.2 (A), Q28.1 (B)
- new net: C40.1, Q24.1 (B), R48.2, R49.1
- new net: D34.1 (K), R49.2
- new net: D30.1 (K), Q20.1 (B)
- new net: C39.1, R43.2, R44.1
- new net: Q23.1 (B), R44.2, R45.1
- new net: D34.2 (A), Q25.3 (C), R50.1
- new net: Q20.3 (C), R40.1
- new net: C37.1, Q19.1 (B), R39.2, R40.2
- new net: R36.1, R37.1, R41.2
- new net: C38.2, Q21.1 (B), Q22.1 (B), R41.1
- new net: Q24.3 (C), Q25.1 (B)
- new net: Q26.2 (E), R51.1
- new net: D33.1 (K), Q24.2 (E)
- new net +24V: Q19.2 (E), Q25.2 (E), Q27.2 (E), Q28.2 (E), R39.1, R42.2, R43.1, R47.1
- new net -24V: R46.1
- new net ADC: R36.2
- new net BDC: R37.2
- new net FAULT: C37.2, D35.1 (K), Q19.3 (C), R38.1
- new net GND: C38.1, C39.2, C40.2, D33.2 (A), Q20.2 (E), Q21.2 (E), Q22.2 (E), Q23.2 (E), R38.2, R51.2
- new net MUT: R50.2
- new net PR: R53.2
- new net PRE1: D32.2 (A), Q26.1 (B), R47.2
- new net TEMP: R52.2
