File: Power Supply Control Board/Power Supply Control Board/Power Supply Control Board SG3525.kicad_sch (KiCad schematic)
At the start: 52 parts, among them J1 Conn_01x14_Male, Q1 BC546, Q2 BC546, Q3 MPSA92, U1 LM393, U2 SG3525, U3 IR2110

Commit message: Finish design of SG3525 Board into SMD
Parts:
- added C14: 100µ/6.3V, Capacitor_Tantalum_SMD:CP_EIA-3528-21_Kemet-B, symbol Device:C_Polarized
- added Q4: MMBT5551L, Package_TO_SOT_SMD:SOT-23, symbol Transistor_BJT:MMBT5551L
- added R28: 10k, Resistor_SMD:R_0805_2012Metric, symbol Device:R
- C1, C13, C4, C5, C7, C8: footprint Capacitor_THT:CP_Radial_D5.0mm_P2.00mm -> Capacitor_SMD:C_0805_2012Metric; LCSC (none) -> C15850
- C10, C2: footprint Capacitor_THT:C_Rect_L7.0mm_W3.5mm_P5.00mm -> Capacitor_SMD:C_0805_2012Metric; LCSC (none) -> C49678
- C11, C9: footprint Capacitor_THT:C_Rect_L7.0mm_W3.5mm_P5.00mm -> Capacitor_SMD:C_0402_1005Metric
- C12: footprint Capacitor_THT:C_Rect_L7.0mm_W3.5mm_P5.00mm -> Capacitor_SMD:C_0402_1005Metric; LCSC (none) -> C1567
- C3: footprint Capacitor_THT:C_Rect_L7.0mm_W3.5mm_P5.00mm -> Capacitor_SMD:C_0402_1005Metric; LCSC (none) -> C1537
- C6: footprint Capacitor_THT:C_Rect_L7.0mm_W3.5mm_P5.00mm -> Capacitor_SMD:C_0402_1005Metric; LCSC (none) -> C15195
- D1: value MURS120 -> US1MG; footprint Diode_THT:D_DO-35_SOD27_P2.54mm_Vertical_AnodeUp -> Diode_SMD:D_SMA; LCSC (none) -> C412437
- D2, D3, D4, D5: footprint Diode_THT:D_DO-35_SOD27_P2.54mm_Vertical_AnodeUp -> Diode_SMD:D_SOD-123; LCSC (none) -> C81598
- Q1, Q2: value BC546 -> MMBT5551L; footprint Package_TO_SOT_THT:TO-92_Inline -> Package_TO_SOT_SMD:SOT-23; symbol Transistor_BJT:BC546 -> Transistor_BJT:MMBT5551L
- Q3: value MPSA92 -> MMBT5401; footprint Package_TO_SOT_THT:TO-92_Inline -> Package_TO_SOT_SMD:SOT-23
- R1, R2, R3: value 150k 0.5W -> 100k 0.5W; footprint Resistor_THT:R_Axial_DIN0309_L9.0mm_D3.2mm_P5.08mm_Vertical -> Resistor_SMD:R_1206_3216Metric
- R10, R11, R12, R13, R15, R17, R18, R19, R20, R21, R22, R23, R24, R25, R27, R5, R6, R7, R8, R9: footprint Resistor_THT:R_Axial_DIN0309_L9.0mm_D3.2mm_P2.54mm_Vertical -> Resistor_SMD:R_0805_2012Metric
- R14: value 10k -> 22k; footprint Resistor_THT:R_Axial_DIN0309_L9.0mm_D3.2mm_P2.54mm_Vertical -> Resistor_SMD:R_0805_2012Metric
- R16: value 10k -> 47k; footprint Resistor_THT:R_Axial_DIN0309_L9.0mm_D3.2mm_P2.54mm_Vertical -> Resistor_SMD:R_0805_2012Metric
- R26: footprint Resistor_THT:R_Axial_DIN0309_L9.0mm_D3.2mm_P2.54mm_Vertical -> Resistor_SMD:R_1206_3216Metric
- R4: value 12k -> 2k7; footprint Resistor_THT:R_Axial_DIN0309_L9.0mm_D3.2mm_P2.54mm_Vertical -> Resistor_SMD:R_0805_2012Metric
- U1: footprint Package_DIP:DIP-8_W7.62mm_LongPads -> Package_SO:SOIC-8_3.9x4.9mm_P1.27mm
- U2: footprint Package_DIP:DIP-16_W7.62mm_Socket_LongPads -> Package_SO:SO-16_3.9x9.9mm_P1.27mm; LCSC (none) -> C68323
- U3: footprint Package_DIP:DIP-14_W7.62mm -> Package_SO:SOIC-16W_7.5x10.3mm_P1.27mm; LCSC (none) -> C2968
Connections:
- net +16V: now also R14.1
- net GND: now also Q1.2 (E), Q2.2 (E), C14.2, Q4.2 (E), R28.2; no longer Q1.3 (E), Q2.3 (E), R14.2
- net ~ShutDown: now also Q2.3 (C); no longer Q2.1 (C)
- net at R10.1, U2.10 (SD): now also Q1.3 (C); no longer Q1.1 (C)
- net at R18.1, R19.1: now also Q2.1 (B); no longer Q2.2 (B)
- net at Q3.3 (C): now also R16.1; no longer R16.2
- new net: C14.1, Q1.1 (B), Q4.3 (C), R14.2
- new net: Q4.1 (B), R16.2, R28.1
Other:
- company: (none) -> Dietmar van Heukelum
- title: (none) -> Power Supply Control Board SG3525
- moved on the sheet: R14
