File: Power Supply Board v2.0/Power Supply Board v2.0.kicad_pcb (KiCad board)
At the start: 2 copper layers, 326 x 150.3 mm, 165 parts, among them J1 CONN_01X03, J10 -BH, J11 CON_AMP_A, J12 CON_AMP_B, J13 CON_LED, J14 CONN_01X03, J2 CON_CTRL_Board, J3 CONN_01X02, J4 CONN_01X02, J5 +BH, J6 G, J7 -BH, J8 +BH, J9 G, K1 Pana JS1-12V-F, Q1 BC546, Q10 BC546, Q11 BC546, Q12 BC546, Q13 BC546, Q14 MPSA56, Q15 BC546, Q16 MPSA06, Q2 MPSA06, Q3 MPSA56, Q4 MPSA06, Q5 MPSA56, Q6 IRFP460, Q7 IRFP460, Q8 MPSA56, Q9 MJE350, T1 Transformer_1P_1S, T3 Half_Bridge_Transformer, U1 LM7815ACT, U2 CNY75G, U3 LM7815ACT, U4 LM7915CT

Commit message: Add Top Layer Zones and some graphics to Main Board V2.0
Parts:
- added REF**: VHAudio_Logo_60mm, LogoLibrary:VHAudio_Logo_60mm, F.Cu at (206.2, 217.6)
Routing:
- net Net-(C13-Pad2): track 165.9 -> 105.6 mm
- net CS-: track 67.0 -> 63.7 mm
- net VB: track 191.1 -> 193.5 mm
- net Net-(C17-Pad1): track 15.8 -> 13.9 mm
- added copper zone on F.Cu, net GND
- added copper zone on F.Cu, net GNDA
- added copper zone on F.Cu, net Net-(C13-Pad2)
Other:
- board text added: "1"
- board text added: "1kW Audio Power Supply"
- board text added: "Control Board"

Commit message: Add stitching and move some components around, so taht they no longer are top of each other
Parts:
- moved C10 60.6 mm to (110.2, 218.4), turned to 90 degrees
- moved HS5 33.0 mm to (93.9, 207.1)
- moved U1 33.0 mm to (91.1, 218.7)
- moved D7 24.2 mm to (103.7, 211.0), turned to -90 degrees
- moved D3 16.1 mm to (61.9, 218.1)
- moved D2 15.9 mm to (61.9, 214.0)
- moved C37 15.8 mm to (277.3, 216.1)
- moved C36 12.1 mm to (263.8, 216.2)
- moved J3 11.2 mm to (335.7, 147.8)
- moved R24 10.6 mm to (243.7, 215.1)
- moved C7 9.46 mm to (48.6, 216.3)
- moved D5 8.60 mm to (73.1, 218.1), turned to 0 degrees
- moved D4 8.55 mm to (73.0, 214.0), turned to 0 degrees
- moved R38 6.61 mm to (312.8, 222.4)
- moved C35 3.52 mm to (283.0, 207.5), turned to 90 degrees
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Routing:
- net +15V: track 143.8 -> 187.4 mm, vias 0 -> 2
- net +16V: track 256.5 -> 230.9 mm
- net /PR2: track 151.6 -> 129.0 mm, vias 0 -> 1
- net Net-(R24-Pad1): track 83.9 -> 73.2 mm
- net HO: track 87.6 -> 77.3 mm, vias 0 -> 1
- net VB: track 193.5 -> 187.4 mm, vias 1 -> 2
- net Net-(C7-Pad1): track 42.8 -> 48.6 mm
- net Net-(C20-Pad1): track 61.5 -> 56.6 mm
- net GNDA: track 199.2 -> 202.6 mm, vias 0 -> 27
- net Net-(D2-Pad2): track 31.5 -> 34.4 mm
- net SIG_B: track 52.9 -> 55.4 mm
- net /PR1: track 98.9 -> 96.6 mm
- net Net-(D3-Pad2): track 54.2 -> 56.4 mm
- net TEMP: track 55.7 -> 57.8 mm
- net -15V: track 121.7 -> 123.7 mm, vias 1 -> 0
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Other:
- board size 326 x 150.3 mm -> 326 x 151 mm
- board text added: "Fan A"
- board text added: "Fan B"
- board text added: "LED Signals"
- board text added: "Power Amp A"
- board text added: "Power Amp B"
- board text added: "Pre Amp Supply"
