File: Auxiliary Power Module/Auxiliary Supply/Auxiliary Supply.kicad_sch (KiCad schematic)
At the start: 19 parts, among them J301 Conn_01x04_Male, J302 Conn_01x04_Male, T1 B66418W1008D1, U301 TNY274P, U302 CNY17-1

Commit message: Finish design of SG3525 Board into SMD
Other:
- title: (none) -> Auxiliary Power Supply Board
Changed lines of the file:
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@@
 (kicad_sch (version 20210126) (generator eeschema)
   (paper "A4")
+  (title_block
+    (title "Auxiliary Power Supply Board")
+    (date "2021-04-07")
+    (rev "V 1.0")
+  )
   (junction (at 100.33 104.775) (diameter 1.016) (color 0 0 0 0))
   (junction (at 101.6 62.865) (diameter 1.016) (color 0 0 0 0))

Commit message: Cleanup of current status for V3.0
Parts:
- C304: footprint Capacitor_THT:CP_Radial_D16.0mm_P7.50mm -> Capacitor_THT:CP_Radial_D6.3mm_P2.50mm
- D301: footprint Diode_SMD:D_SMB -> Diode_SMD:D_SMB_Handsoldering
- D304: value BZX84C15 -> BZX85C12; footprint Diode_SMD:D_SOT-23_ANK -> Diode_THT:D_DO-41_SOD81_P3.81mm_Vertical_KathodeUp
Other:
- moved on the sheet: J302
Changed lines of the file:
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@@
   (junction (at 133.985 90.805) (diameter 1.016) (color 0 0 0 0))
   (junction (at 149.225 111.125) (diameter 1.016) (color 0 0 0 0))
+  (junction (at 161.925 38.735) (diameter 1.016) (color 0 0 0 0))
   (junction (at 161.925 52.705) (diameter 1.016) (color 0 0 0 0))
   (junction (at 161.925 73.025) (diameter 1.016) (color 0 0 0 0))
@@
   (junction (at 178.435 98.425) (diameter 1.016) (color 0 0 0 0))
   (junction (at 178.435 111.125) (diameter 1.016) (color 0 0 0 0))
-  (junction (at 194.31 106.045) (diameter 1.016) (color 0 0 0 0))
-  (junction (at 201.93 106.045) (diameter 1.016) (color 0 0 0 0))
+  (junction (at 201.93 111.125) (diameter 1.016) (color 0 0 0 0))
   (no_connect (at 97.79 99.695))
   (no_connect (at 97.79 102.235))
   (no_connect (at 159.385 98.425))
-  (no_connect (at 203.835 100.965))
-  (no_connect (at 203.835 103.505))
+  (no_connect (at 203.835 106.045))
+  (no_connect (at 203.835 108.585))
   (wire (pts (xy 97.79 97.155) (xy 103.505 97.155))
     (stroke (width 0) (type solid) (color 0 0 0 0))
@@
     (stroke (width 0) (type solid) (color 0 0 0 0))
   )
+  (wire (pts (xy 161.925 37.465) (xy 161.925 38.735))
+    (stroke (width 0) (type solid) (color 0 0 0 0))
+  )
   (wire (pts (xy 161.925 38.735) (xy 161.925 52.705))
     (stroke (width 0) (type solid) (color 0 0 0 0))
@@
     (stroke (width 0) (type solid) (color 0 0 0 0))
   )
-  (wire (pts (xy 178.435 111.125) (xy 194.31 111.125))
-    (stroke (width 0) (type solid) (color 0 0 0 0))
-  )
-  (wire (pts (xy 194.31 106.045) (xy 201.93 106.045))
-    (stroke (width 0) (type solid) (color 0 0 0 0))
-  )
-  (wire (pts (xy 194.31 111.125) (xy 194.31 106.045))
-    (stroke (width 0) (type solid) (color 0 0 0 0))
-  )
-  (wire (pts (xy 198.755 98.425) (xy 203.835 98.425))
-    (stroke (width 0) (type solid) (color 0 0 0 0))
-  )
-  (wire (pts (xy 201.93 106.045) (xy 201.93 108.585))
-    (stroke (width 0) (type solid) (color 0 0 0 0))
-  )
-  (wire (pts (xy 203.835 106.045) (xy 201.93 106.045))
+  (wire (pts (xy 178.435 111.125) (xy 201.93 111.125))
+    (stroke (width 0) (type solid) (color 0 0 0 0))
+  )
+  (wire (pts (xy 198.755 103.505) (xy 203.835 103.505))
+    (stroke (width 0) (type solid) (color 0 0 0 0))
+  )
+  (wire (pts (xy 201.93 111.125) (xy 201.93 113.665))
+    (stroke (width 0) (type solid) (color 0 0 0 0))
+  )
+  (wire (pts (xy 203.835 111.125) (xy 201.93 111.125))
     (stroke (width 0) (type solid) (color 0 0 0 0))
   )
@@
     )
   )
-  (global_label "+Vcc" (shape input) (at 198.755 98.425 180)
+  (global_label "+Vcc" (shape input) (at 198.755 103.505 180)
     (effects (font (size 1.27 1.27)) (justify right))
-    (property "Intersheet References" "${INTERSHEET_REFS}" (id 0) (at 73.025 247.015 0)
+    (property "Intersheet References" "${INTERSHEET_REFS}" (id 0) (at 73.025 252.095 0)
       (effects (font (size 1.27 1.27)) hide)
     )
@@
     (pin "1")
   )
-  (symbol (lib_id "power:PWR_FLAG") (at 194.31 106.045 0) (unit 1)
-    (in_bom yes) (on_board yes)
-    (property "Reference" "#FLG0101" (id 0) (at 194.31 104.14 0)
-      (effects (font (size 1.27 1.27)) hide)
-    )
-    (property "Value" "PWR_FLAG" (id 1) (at 194.31 101.7206 0)
-      (effects (font (size 1.27 1.27)) hide)
-    )
-    (property "Footprint" "" (id 2) (at 194.31 106.045 0)
-      (effects (font (size 1.27 1.27)) hide)
-    )
-    (property "Datasheet" "~" (id 3) (at 194.31 106.045 0)
+  (symbol (lib_id "power:PWR_FLAG") (at 161.925 37.465 0) (unit 1)
+    (in_bom yes) (on_board yes)
+    (property "Reference" "#FLG0101" (id 0) (at 161.925 35.56 0)
+      (effects (font (size 1.27 1.27)) hide)
+    )
+    (property "Value" "PWR_FLAG" (id 1) (at 161.925 33.1406 0)
+      (effects (font (size 1.27 1.27)) hide)
+    )
+    (property "Footprint" "" (id 2) (at 161.925 37.465 0)
+      (effects (font (size 1.27 1.27)) hide)
+    )
+    (property "Datasheet" "~" (id 3) (at 161.925 37.465 0)
       (effects (font (size 1.27 1.27)) hide)
     )
@@
     (pin "1")
   )
-  (symbol (lib_id "power:GND") (at 201.93 108.585 0) (unit 1)
-    (in_bom yes) (on_board yes)
-    (property "Reference" "#PWR0303" (id 0) (at 201.93 114.935 0)
-      (effects (font (size 1.27 1.27)) hide)
-    )
-    (property "Value" "GND" (id 1) (at 202.057 112.9792 0))
-    (property "Footprint" "" (id 2) (at 201.93 108.585 0)
-      (effects (font (size 1.27 1.27)) hide)
-    )
-    (property "Datasheet" "" (id 3) (at 201.93 108.585 0)
+  (symbol (lib_id "power:GND") (at 201.93 113.665 0) (unit 1)
+    (in_bom yes) (on_board yes)
+    (property "Reference" "#PWR0303" (id 0) (at 201.93 120.015 0)
+      (effects (font (size 1.27 1.27)) hide)
+    )
+    (property "Value" "GND" (id 1) (at 202.057 118.0592 0))
+    (property "Footprint" "" (id 2) (at 201.93 113.665 0)
+      (effects (font (size 1.27 1.27)) hide)
+    )
+    (property "Datasheet" "" (id 3) (at 201.93 113.665 0)
       (effects (font (size 1.27 1.27)) hide)
     )
@@
       (effects (font (size 1.27 1.27)) (justify right))
     )
-    (property "Footprint" "Diode_SMD:D_SMB" (id 2) (at 127.635 67.31 0)
+    (property "Footprint" "Diode_SMD:D_SMB_Handsoldering" (id 2) (at 127.635 67.31 0)
       (effects (font (size 1.27 1.27)) hide)
     )
@@
       (effects (font (size 1.27 1.27)) (justify left))
     )
-    (property "Value" "BZX84C15" (id 1) (at 180.467 81.788 90)
-      (effects (font (size 1.27 1.27)) (justify left))
-    )
-    (property "Footprint" "Diode_SMD:D_SOT-23_ANK" (id 2) (at 173.99 80.645 0)
+    (property "Value" "BZX85C12" (id 1) (at 180.467 81.788 90)
+      (effects (font (size 1.27 1.27)) (justify left))
+    )
+    (property "Footprint" "Diode_THT:D_DO-41_SOD81_P3.81mm_Vertical_KathodeUp" (id 2) (at 173.99 80.645 0)
       (effects (font (size 1.27 1.27)) hide)
     )
@@
       (effects (font (size 1.27 1.27)) (justify left))
     )
-    (property "Footprint" "Capacitor_THT:CP_Radial_D16.0mm_P7.50mm" (id 2) (at 173.0502 72.39 0)
+    (property "Footprint" "Capacitor_THT:CP_Radial_D6.3mm_P2.50mm" (id 2) (at 173.0502 72.39 0)
       (effects (font (size 1.27 1.27)) hide)
     )
@@
     (pin "4")
   )
-  (symbol (lib_id "Connector:Conn_01x04_Male") (at 208.915 100.965 0) (mirror y) (unit 1)
-    (in_bom yes) (on_board yes)
-    (property "Reference" "J302" (id 0) (at 203.276 94.659 0)
+  (symbol (lib_id "Connector:Conn_01x04_Male") (at 208.915 106.045 0) (mirror y) (unit 1)
+    (in_bom yes) (on_board yes)
+    (property "Reference" "J302" (id 0) (at 203.276 99.739 0)
       (effects (font (size 1.27 1.27)) (justify right))
     )
-    (property "Value" "Conn_01x04_Male" (id 1) (at 209.6263 103.9431 0)
+    (property "Value" "Conn_01x04_Male" (id 1) (at 209.6263 109.0231 0)
       (effects (font (size 1.27 1.27)) (justify right) hide)
     )
-    (property "Footprint" "Connector_PinHeader_2.54mm:PinHeader_1x04_P2.54mm_Vertical" (id 2) (at 208.915 100.965 0)
-      (effects (font (size 1.27 1.27)) hide)
-    )
-    (property "Datasheet" "~" (id 3) (at 208.915 100.965 0)
+    (property "Footprint" "Connector_PinHeader_2.54mm:PinHeader_1x04_P2.54mm_Vertical" (id 2) (at 208.915 106.045 0)
+      (effects (font (size 1.27 1.27)) hide)
+    )
+    (property "Datasheet" "~" (id 3) (at 208.915 106.045 0)
       (effects (font (size 1.27 1.27)) hide)
     )
@@
     )
     (path "/00000000-0000-0000-0000-00005edb2db8"
-      (reference "C304") (unit 1) (value "120µ 20V") (footprint "Capacitor_THT:CP_Radial_D16.0mm_P7.50mm")
+      (reference "C304") (unit 1) (value "120µ 20V") (footprint "Capacitor_THT:CP_Radial_D6.3mm_P2.50mm")
     )
     (path "/100faac4-b4f2-480f-b3d2-9e45153b5642"
@@
     )
     (path "/9fa82c58-d5fc-48f6-bc77-95db5252b2a4"
-      (reference "D301") (unit 1) (value "SM6T150A") (footprint "Diode_SMD:D_SMB")
+      (reference "D301") (unit 1) (value "SM6T150A") (footprint "Diode_SMD:D_SMB_Handsoldering")
     )
     (path "/00000000-0000-0000-0000-00005edab524"
@@
     )
     (path "/00000000-0000-0000-0000-00005edb1bdc"
-      (reference "D304") (unit 1) (value "BZX84C15") (footprint "Diode_SMD:D_SOT-23_ANK")
+      (reference "D304") (unit 1) (value "BZX85C12") (footprint "Diode_THT:D_DO-41_SOD81_P3.81mm_Vertical_KathodeUp")
     )
     (path "/b0e092e8-6a7f-482f-935f-be31cf6e25a2"
